File: pcb/morningtown.kicad_pcb (KiCad board)
At the start: 2 copper layers, 30 x 95 mm, 13 parts, among them SW1 Test, U1 Pico, U2 DS3231M

Commit message: Work on PCB
Parts:
- added R4: 4.7k, Resistor_SMD:R_0805_2012Metric_Pad1.20x1.40mm_HandSolder, F.Cu at (126.5, 115.5)
- added R5: 4.7k, Resistor_SMD:R_0805_2012Metric_Pad1.20x1.40mm_HandSolder, F.Cu at (126.5, 118.5)
Routing:
- net Net-(U1-GPIO4): track 64.0 -> 80.0 mm, vias 0 -> 2
- net Net-(U1-VSYS): track 78.6 -> 85.7 mm
- net Net-(U1-GPIO5): track 54.2 -> 59.6 mm
- net Net-(U1-GPIO6): vias 1 -> 3
