File: pcb/morningtown.kicad_sch (KiCad schematic)
At the start: 11 parts, among them SW1 Test, U1 Pico, U2 DS3231M

Commit message: Update KiCad files to latest version, update errata, add metadata
Other:
- company: (none) -> https://www.bitwiz.me.uk/
- title: (none) -> MorningTown
Changed lines of the file:
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@@
 (kicad_sch
-	(version 20231120)
+	(version 20250114)
 	(generator "eeschema")
-	(generator_version "8.0")
+	(generator_version "9.0")
 	(paper "A4")
+	(title_block
+		(title "MorningTown")
+		(date "2026-03-15")
+		(rev "1.2")
+		(company "https://www.bitwiz.me.uk/")
+		(comment 1 "https://github.com/taw10/morningtown")
+	)
 	(junction
 		(at 66.04 58.42)
@@
 		)
 	)
+	(embedded_fonts no)
 )

Commit message: Work on PCB
Parts:
- added R4, R5: 4.7k, Resistor_SMD:R_0805_2012Metric_Pad1.20x1.40mm_HandSolder, symbol Device:R
- D3, R3: now not fitted
Connections:
- net at C2.1, U1.39 (VSYS), U2.2 (VCC): now also R4.1, R5.1
- net at U1.6 (GPIO4), U2.7 (SDA): now also R4.2
- net at U1.7 (GPIO5), U2.8 (SCL): now also R5.2
Changed lines of the file:
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@@
 	)
 	(junction
-		(at 66.04 58.42)
+		(at 66.04 55.88)
 		(diameter 0)
 		(color 0 0 0 0)
@@
 	)
 	(junction
+		(at 71.12 63.5)
+		(diameter 0)
+		(color 0 0 0 0)
+	)
+	(junction
+		(at 71.12 55.88)
+		(diameter 0)
+		(color 0 0 0 0)
+	)
+	(junction
 		(at 143.51 135.89)
 		(diameter 0)
@@
 	)
 	(junction
+		(at 77.47 66.04)
+		(diameter 0)
+		(color 0 0 0 0)
+	)
+	(junction
 		(at 121.92 116.84)
 		(diameter 0)
@@
 	)
 	(junction
+		(at 77.47 55.88)
+		(diameter 0)
+		(color 0 0 0 0)
+	)
+	(junction
 		(at 80.01 135.89)
 		(diameter 0)
@@
 	(wire
 		(pts
-			(xy 74.93 63.5) (xy 74.93 88.9)
+			(xy 71.12 63.5) (xy 71.12 88.9)
 		)
 		(stroke
@@
 	(wire
 		(pts
-			(xy 127 58.42) (xy 127 76.2)
+			(xy 127 55.88) (xy 127 76.2)
 		)
 		(stroke
@@
 	(wire
 		(pts
-			(xy 66.04 58.42) (xy 66.04 69.85)
-		)
-		(stroke
-			(width 0)
-			(type default)
-		)
-	)
-	(wire
-		(pts
 			(xy 118.11 104.14) (xy 121.92 104.14)
 		)
@@
 	(wire
 		(pts
+			(xy 66.04 55.88) (xy 71.12 55.88)
+		)
+		(stroke
+			(width 0)
+			(type default)
+		)
+	)
+	(wire
+		(pts
 			(xy 80.01 116.84) (xy 80.01 135.89)
 		)
@@
 	(wire
 		(pts
-			(xy 82.55 88.9) (xy 74.93 88.9)
-		)
-		(stroke
-			(width 0)
-			(type default)
-		)
-	)
-	(wire
-		(pts
-			(xy 66.04 58.42) (xy 55.88 58.42)
+			(xy 82.55 88.9) (xy 71.12 88.9)
 		)
 		(stroke
@@
 	(wire
 		(pts
-			(xy 66.04 58.42) (xy 127 58.42)
-		)
-		(stroke
-			(width 0)
-			(type default)
-		)
-	)
-	(wire
-		(pts
 			(xy 80.01 135.89) (xy 121.92 135.89)
 		)
@@
 	(wire
 		(pts
-			(xy 55.88 58.42) (xy 55.88 55.88)
-		)
-		(stroke
-			(width 0)
-			(type default)
-		)
-	)
-	(wire
-		(pts
 			(xy 49.53 55.88) (xy 49.53 58.42)
 		)
@@
 	(wire
 		(pts
+			(xy 77.47 55.88) (xy 77.47 58.42)
+		)
+		(stroke
+			(width 0)
+			(type default)
+		)
+	)
+	(wire
+		(pts
 			(xy 49.53 135.89) (xy 80.01 135.89)
 		)
@@
 	(wire
 		(pts
-			(xy 55.88 55.88) (xy 49.53 55.88)
+			(xy 49.53 55.88) (xy 66.04 55.88)
 		)
 		(stroke
@@
 	(wire
 		(pts
+			(xy 71.12 55.88) (xy 77.47 55.88)
+		)
+		(stroke
+			(width 0)
+			(type default)
+		)
+	)
+	(wire
+		(pts
 			(xy 158.75 101.6) (xy 158.75 106.68)
 		)
@@
 	(wire
 		(pts
+			(xy 77.47 55.88) (xy 127 55.88)
+		)
+		(stroke
+			(width 0)
+			(type default)
+		)
+	)
+	(wire
+		(pts
 			(xy 49.53 80.01) (xy 49.53 85.09)
 		)
@@
 	(wire
 		(pts
+			(xy 66.04 55.88) (xy 66.04 69.85)
+		)
+		(stroke
+			(width 0)
+			(type default)
+		)
+	)
+	(wire
+		(pts
 			(xy 82.55 116.84) (xy 80.01 116.84)
 		)
@@
 	(wire
 		(pts
-			(xy 62.23 63.5) (xy 74.93 63.5)
+			(xy 62.23 63.5) (xy 71.12 63.5)
 		)
 		(stroke
@@
 		(in_bom yes)
 		(on_board yes)
-		(dnp no)
+		(dnp yes)
 		(property "Reference" "R3"
 			(at 143.002 105.41 90)
@@
 				(path "/89214f91-96ed-4d86-ae81-f3a706929ffe"
 					(reference "R2")
+					(unit 1)
+				)
+			)
+		)
+	)
+	(symbol
+		(lib_id "Device:R")
+		(at 71.12 59.69 0)
+		(unit 1)
+		(exclude_from_sim no)
+		(in_bom yes)
+		(on_board yes)
+		(dnp no)
+		(fields_autoplaced yes)
+		(property "Reference" "R5"
+			(at 73.66 58.4199 0)
+			(effects
+				(font
+					(size 1.27 1.27)
+				)
+				(justify left)
+			)
+		)
+		(property "Value" "4.7k"
+			(at 73.66 60.9599 0)
+			(effects
+				(font
+					(size 1.27 1.27)
+				)
+				(justify left)
+			)
+		)
+		(property "Footprint" "Resistor_SMD:R_0805_2012Metric_Pad1.20x1.40mm_HandSolder"
+			(at 69.342 59.69 90)
+			(effects
+				(font
+					(size 1.27 1.27)
+				)
+				(hide yes)
+			)
+		)
+		(property "Datasheet" "~"
+			(at 71.12 59.69 0)
+			(effects
+				(font
+					(size 1.27 1.27)
+				)
+				(hide yes)
+			)
+		)
+		(property "Description" "Resistor"
+			(at 71.12 59.69 0)
+			(effects
+				(font
+					(size 1.27 1.27)
+				)
+				(hide yes)
+			)
+		)
+		(pin "1"
+		)
+		(pin "2"
+		)
+		(instances
+			(project ""
+				(path "/89214f91-96ed-4d86-ae81-f3a706929ffe"
+					(reference "R5")
 					(unit 1)
 				)
@@
 	)
 	(symbol
+		(lib_id "Device:R")
+		(at 77.47 62.23 0)
+		(unit 1)
+		(exclude_from_sim no)
+		(in_bom yes)
+		(on_board yes)
+		(dnp no)
+		(fields_autoplaced yes)
+		(property "Reference" "R4"
+			(at 80.01 60.9599 0)
+			(effects
+				(font
+					(size 1.27 1.27)
+				)
+				(justify left)
+			)
+		)
+		(property "Value" "4.7k"
+			(at 80.01 63.4999 0)
+			(effects
+				(font
+					(size 1.27 1.27)
+				)
+				(justify left)
+			)
+		)
+		(property "Footprint" "Resistor_SMD:R_0805_2012Metric_Pad1.20x1.40mm_HandSolder"
+			(at 75.692 62.23 90)
+			(effects
+				(font
+					(size 1.27 1.27)
+				)
+				(hide yes)
+			)
+		)
+		(property "Datasheet" "~"
+			(at 77.47 62.23 0)
+			(effects
+				(font
+					(size 1.27 1.27)
+				)
+				(hide yes)
+			)
+		)
+		(property "Description" "Resistor"
+			(at 77.47 62.23 0)
+			(effects
+				(font
+					(size 1.27 1.27)
+				)
+				(hide yes)
+			)
+		)
+		(pin "2"
+		)
+		(pin "1"
+		)
+		(instances
+			(project ""
+				(path "/89214f91-96ed-4d86-ae81-f3a706929ffe"
+					(reference "R4")
+					(unit 1)
+				)
+			)
+		)
+	)
+	(symbol
 		(lib_id "Timer_RTC:DS3231MZ")
 		(at 49.53 68.58 0)
@@
 		(in_bom yes)
 		(on_board yes)
-		(dnp no)
+		(dnp yes)
 		(property "Reference" "D3"
 			(at 162.814 105.41 0)
